File: hardware/LoRaModule.sch (KiCad schematic (older format))
At the start: 28 parts, among them J1 Conn_Coaxial, J3 Screw_Terminal_01x02, J4 Screw_Terminal_01x03, J6 Screw_Terminal_01x03, M1 DC-DC_Buck_Step_Module, SW1 SW_DIP_x01, U1 RFM95W-868S2, U2 ARDUINO_Pro-MiniALL

Commit message: Update the hardware design files
Other:
- note added: "1.0"
- note added: "2020/09/10"
- note added: "AGRIOT LoRa Sensor"
- note removed: "Alimentación arduino , es necesario más de 3.3v por raw"
- note removed: "Añadir botón de reset y configuration mode"
- note removed: "Falta pull-up en bus de sensor"
- note removed: "¿pull-up en chip select de spi?"
- moved on the sheet: +3V3, A2, A3, A6, A7, C1, D1, DIO1, DIO2, DIO3, DIO5, GND1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

Commit message: Update hardware schematic
Other:
- note removed: "1.0"
- note removed: "2020/09/10"
- note removed: "AGRIOT LoRa Sensor"
Changed lines of the file:
@@
 encoding utf-8
 Sheet 1 1
-Title ""
-Date ""
-Rev ""
+Title "AGRIOT LoRa Sensor"
+Date "2020-09-10"
+Rev "1.0"
 Comp ""
 Comment1 ""
@@
 	1    0    0    -1
 $EndComp
-Text Notes 7400 7500 0    50   ~ 0
-AGRIOT LoRa Sensor
-Text Notes 10600 7650 0    50   ~ 0
-1.0
-Text Notes 8100 7650 0    50   ~ 0
-2020/09/10
 Wire Wire Line
 	1650 4650 2000 4650
